File: controller-pcb/controller/controller.kicad_pcb (KiCad board)
At the start: 2 copper layers, 20 parts, among them J1 Conn_01x04, J10 Conn_01x04, J11 Conn_01x04, J12 Conn_01x04, J13 Conn_01x04, J14 Conn_01x04, J15 Conn_01x04, J16 Conn_01x04, J17 Conn_01x04, J18 Conn_01x04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

Commit message: preparing for Production
Routing:
- net Net-(J4-Pin_2): track 0.00 -> 54.5 mm
- net Net-(J9-Pin_2): track 0.00 -> 48.3 mm
- net Net-(J10-Pin_2): track 0.00 -> 46.7 mm
- net Net-(J9-Pin_3): track 0.00 -> 43.9 mm
- net Net-(A1-D50_MISO): track 0.00 -> 40.3 mm
- net Net-(J9-Pin_4): track 0.00 -> 39.5 mm
- net Net-(A1-D51_MOSI): track 0.00 -> 38.7 mm
- net Net-(J5-Pin_2): track 0.00 -> 22.4 mm
- net Net-(J2-Pin_2): track 0.00 -> 21.1 mm
- net Net-(J6-Pin_3): track 0.00 -> 20.8 mm
- net Net-(J1-Pin_2): track 0.00 -> 20.1 mm
- net Net-(J17-Pin_4): track 0.00 -> 19.4 mm
- net Net-(J3-Pin_2): track 0.00 -> 18.8 mm
- net Net-(J15-Pin_4): track 0.00 -> 18.5 mm
- net Net-(J2-Pin_3): track 0.00 -> 18.3 mm
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Other:
- board outline added: 70 x 60 mm
